File: Source/BUZZER.kicad_pcb (KiCad board)
At the start: 2 copper layers, 63.1 x 95 mm, 22 parts, among them IC1 LM556, J1 USB_A, U1 4017

Commit message: Add Files
Parts:
- added C6: 100nF, Capacitor_THT:C_Disc_D8.0mm_W5.0mm_P5.00mm, F.Cu at (139.5, 104.0)
- added C7: 100uF, Capacitor_THT:C_Radial_D5.0mm_H11.0mm_P2.00mm, F.Cu at (141.0, 111.2)
- C1, C2: value 10nF -> 10uF
- moved R2 7.84 mm to (138.2, 116.6)
- moved R3 6.13 mm to (138.2, 121.1)
- moved C1 1.25 mm to (152.9, 84.7)
- moved C2 0.10 mm to (152.9, 94.8)
Connections:
- C1 pad 1: Net-(IC1-TRES1) -> Net-(C1-Pad1)
- C2 pad 1: Net-(IC1-TRES2) -> GND
- C2 pad 2: GND -> Net-(C2-Pad2)
- IC1 pad 12: Net-(IC1-TRES2) -> GND
- IC1 pad 2: Net-(IC1-TRES1) -> GND
- IC1 pad 6: Net-(IC1-TRES1) -> GND
- IC1 pad 8: Net-(IC1-TRES2) -> GND
- RV1 pad 2: Net-(IC1-TRES1) -> Net-(C1-Pad1)
- RV1 pad 3: Net-(IC1-TRES1) -> GND
- RV2 pad 2: Net-(IC1-TRES2) -> Net-(C2-Pad2)
- RV2 pad 3: Net-(IC1-TRES2) -> GND
Routing:
- net Net-(IC1-TRES2): track 89.6 -> 0.00 mm
- net Net-(IC1-TRES1): track 75.4 -> 0.00 mm
- net Net-(C1-Pad1): track 0.00 -> 48.1 mm
- net Net-(C2-Pad2): track 0.00 -> 47.3 mm
- net GND: track 0.00 -> 29.2 mm
- net OUT 2: track 198.3 -> 206.8 mm
- net VCC: track 88.6 -> 83.7 mm
- net Net-(IC1-DIS1): track 68.2 -> 64.8 mm
- net Net-(IC1-DIS2): track 50.7 -> 49.6 mm
Other:
- outline, holes or cut-outs redrawn
