File: Source/BUZZER.kicad_sch (KiCad schematic)
At the start: 21 parts, among them IC1 LM556, J1 USB_A, U1 4017

Commit message: Add Files
Parts:
- added C6: 100nF, Capacitor_THT:C_Disc_D8.0mm_W5.0mm_P5.00mm, symbol Device:C_Small
- added C7: 100uF, Capacitor_THT:C_Radial_D5.0mm_H11.0mm_P2.00mm, symbol Device:C_Polarized_Small
- C1, C2: value 10nF -> 10uF
Connections:
- net GND: now also C2.1, IC1.12 (TRES2), IC1.2 (TRES1), IC1.6 (TRIG1), IC1.8 (TRIG2), RV1.3, RV2.3, C6.2, C7.2; no longer C2.2
- net VCC: now also C6.1, C7.1
- new net: C1.1, RV1.2
- new net: C2.2, RV2.2
Other:
- moved on the sheet: J1
